File: AeroBlinker.kicad_sch (KiCad schematic)
At the start: 34 parts, among them J1 LED_GND, J2 LED_GND, J3 LED_GND, J4 BATTERY, J5 RECEIVER, J6 USB_C_Receptacle_USB2.0_16P, Q1 AO3400A, SW2 SW_Push, U1 STM32F042F6Px, U2 USBLC6-2SC6, U3 TPS62162DGR

Commit message: Autosave
Connections:
- net USB_D+: no longer U2.6 (I/O1)
Changed lines of the file:
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@@
-		)
-	)
-	(label "USB_D+"
-		(at 160.02 60.96 0)
-		(effects
-			(font
-				(size 1.27 1.27)
-			)
-			(justify left bottom)
 		)
 	)
@@
 		(effects
 			(font
+				(size 1.27 1.27)
+			)
+			(justify left bottom)
+		)
+	)
+	(label "USB_D+"
+		(at 161.29 67.31 0)
+		(effects
+			(font

Commit message: SCH Save
Connections:
- net USB_D+: now also U2.4 (I/O2)
- net USB_D-: now also U2.6 (I/O1); no longer U2.4 (I/O2)
Changed lines of the file:
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@@
-		)
-	)
-	(label "USB_D-"
-		(at 160.02 63.5 0)
-		(effects
-			(font
-				(size 1.27 1.27)
-			)
-			(justify left bottom)
 		)
 	)
@@
 	)
 	(label "USB_D+"
-		(at 161.29 67.31 0)
+		(at 160.02 63.5 0)
 		(effects
 			(font
@@
 		)
 	)
+	(label "USB_D-"
+		(at 160.02 60.96 0)
+		(effects
+			(font
+				(size 1.27 1.27)
+			)
+			(justify left bottom)
+		)
+	)

Commit message: Autosave
Parts:
- U3: footprint Package_SON:Texas_DSG0008A_WSON-8-1EP_2x2mm_P0.5mm_EP0.9x1.6mm_ThermalVias -> Package_SON:Texas_DSG0008A_WSON-8-1EP_2x2mm_P0.5mm_EP0.9x1.6mm
Changed lines of the file:
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@@
 			)
 		)
-		(property "Footprint" "Package_SON:Texas_DSG0008A_WSON-8-1EP_2x2mm_P0.5mm_EP0.9x1.6mm_ThermalVias"
+		(property "Footprint" "Package_SON:Texas_DSG0008A_WSON-8-1EP_2x2mm_P0.5mm_EP0.9x1.6mm"
 			(at 64.77 138.43 0)
 			(hide yes)

Commit message: Autosave
Parts:
- TP2: footprint TestPoint:TestPoint_2Pads_Pitch5.08mm_Drill1.3mm -> TestPoint:TestPoint_Pad_1.0x1.0mm
Changed lines of the file:
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@@
 			)
 		)
-		(property "Footprint" "TestPoint:TestPoint_2Pads_Pitch5.08mm_Drill1.3mm"
+		(property "Footprint" "TestPoint:TestPoint_Pad_1.0x1.0mm"
 			(at 114.3 86.36 0)
 			(hide yes)

Commit message: Autosave
Parts:
- TP1: footprint TestPoint:TestPoint_2Pads_Pitch5.08mm_Drill1.3mm -> TestPoint:TestPoint_Pad_1.0x1.0mm
Changed lines of the file:
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@@
 			)
 		)
-		(property "Footprint" "TestPoint:TestPoint_2Pads_Pitch5.08mm_Drill1.3mm"
+		(property "Footprint" "TestPoint:TestPoint_Pad_1.0x1.0mm"
 			(at 114.3 88.9 0)
 			(hide yes)

Commit message: Autosave
Parts:
- TP2: footprint TestPoint:TestPoint_Pad_1.0x1.0mm -> TestPoint:TestPoint_Pad_1.5x1.5mm
Changed lines of the file:
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@@
 			)
 		)
-		(property "Footprint" "TestPoint:TestPoint_Pad_1.0x1.0mm"
+		(property "Footprint" "TestPoint:TestPoint_Pad_1.5x1.5mm"
 			(at 114.3 86.36 0)
 			(hide yes)

Commit message: Autosave
Parts:
- TP1: footprint TestPoint:TestPoint_Pad_1.0x1.0mm -> TestPoint:TestPoint_Pad_1.5x1.5mm
Changed lines of the file:
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@@
 			)
 		)
-		(property "Footprint" "TestPoint:TestPoint_Pad_1.0x1.0mm"
+		(property "Footprint" "TestPoint:TestPoint_Pad_1.5x1.5mm"
 			(at 114.3 88.9 0)
 			(hide yes)

Commit message: Autosave
Parts:
- renumbered TP2 to TP1, TP1 to TP2
Changed lines of the file:
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@@
 		(in_pos_files yes)
 		(dnp no)
-		(property "Reference" "TP1"
+		(property "Reference" "TP2"
 			(at 118.618 83.82 90)
 			(show_name no)
@@
 			(project "AeroBlinker"
 				(path "/bec00f4f-4b10-4354-9a48-d4013e030360"
-					(reference "TP1")
+					(reference "TP2")
 					(unit 1)
 				)
@@
 		(in_pos_files yes)
 		(dnp no)
-		(property "Reference" "TP2"
+		(property "Reference" "TP1"
 			(at 118.618 81.28 90)
 			(show_name no)
@@
 			(project "AeroBlinker"
 				(path "/bec00f4f-4b10-4354-9a48-d4013e030360"
-					(reference "TP2")
+					(reference "TP1")
 					(unit 1)
 				)
