File: AeroBlinker_WITH_VDDA.kicad_sch (KiCad schematic)
At the start: 34 parts, among them J1 LED_GND, J2 LED_GND, J3 LED_GND, J4 BATTERY, J5 RECEIVER, J6 USB_C_Receptacle_USB2.0_16P, Q1 AO3400A, SW2 SW_Push, U1 STM32F042F6Px, U2 USBLC6-2SC6, U3 TPS62160DSG

Commit message: Pre-restore backup: 5 files changed AeroBlinker.kicad_pcb 0/40/495 AeroBlinker.kicad_prl 127/0/0 AeroBlinker.kicad_pro 701/0/0 AeroBlinker.kicad_sch 98/0/248 AeroBlinker_WITH_VDDA.kicad_sch 10901/0/0
Parts:
- removed D2: BZT585B3V3T-7, Package_TO_SOT_SMD:SOT-23, symbol Diode:BZX84Cxx
- removed J5: RECEIVER, Connector_JST:JST_VH_B2P-VH_1x02_P3.96mm_Vertical, symbol Connector_Generic:Conn_01x02
- removed R6: 1K, Resistor_SMD:R_0402_1005Metric, symbol Device:R
- C1, C4, C6: footprint Capacitor_SMD:C_0402_1005Metric -> Package_SON:WSON-6-1EP_2x2mm_P0.65mm_EP1x1.6mm_ThermalVias
- C2: footprint Capacitor_SMD:C_0603_1608Metric -> (none)
- C3, C5: footprint Capacitor_SMD:C_0402_1005Metric -> (none)
- C7, C9: footprint Capacitor_SMD:C_0603_1608Metric -> Package_SON:WSON-6-1EP_2x2mm_P0.65mm_EP1x1.6mm_ThermalVias
- FB1: footprint Inductor_SMD:L_0603_1608Metric -> (none)
- H1, H2, H3, H4: footprint MountingHole:MountingHole_2.1mm -> (none)
- J1: renamed from J6; footprint Connector_USB:USB_C_Receptacle_GCT_USB4105-xx-A_16P_TopMnt_Horizontal -> (none)
- L1: footprint Inductor_SMD:L_Changjiang_FNR3012S -> Package_SON:Texas_DSG0008A_WSON-8-1EP_2x2mm_P0.5mm_EP0.9x1.6mm_ThermalVias
- R1, R2, R3, R4, R5: footprint Resistor_SMD:R_0402_1005Metric -> Package_DIP:DIP-8_W7.62mm
- SW2: footprint Button_Switch_THT:SW_PUSH_1P1T_6x3.5mm_H4.3_APEM_MJTP1243 -> Button_Switch_SMD:Nidec_Copal_CAS-120A
- renumbered TP2 to TP1
Connections:
- net BOOT: now also R1.2, SW2.2
- net RECV_PWM renamed TIM2_CH1
- no-connect marks 11 -> 9
Other:
- note removed: "Receiver In"
- moved on the sheet: C1, C2, C3, C4, C5, C6, FB1, H1, H2, H3, H4, R1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
