File: AeroBlinker.kicad_pcb (KiCad board)
At the start: 2 copper layers, 41.8 x 28 mm, 33 parts, among them J1 LED_GND, J2 LED_GND, J3 LED_GND, J4 BATTERY, J5 RECEIVER, J6 USB_C_Receptacle_USB2.0_16P, Q1 AO3400A, SW2 SW_Push, U1 STM32F042F6Px, U2 USBLC6-2SC6, U3 TPS62162DGR

Commit message: Autosave
Parts:
- moved R6 1.61 mm to (144.8, 126.2)
- moved R1 1.61 mm to (144.7, 125.0)
Changed lines of the file:
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@@
 	(footprint "Resistor_SMD:R_0402_1005Metric"
 		(layer "F.Cu")
-		(at 146.3525 124.925)
+		(at 144.74 125)
 		(descr "Resistor SMD 0402 (1005 Metric), square (rectangular) end terminal, IPC-7351 nominal, (Body size source: IPC-SM-782 page 72, https://www.pcb-3d.com/wordpress/wp-content/uploads/ipc-sm-782a_amendment_1_and_2.pdf)")
 		(tags "resistor")
@@
 	(footprint "Resistor_SMD:R_0402_1005Metric"
 		(layer "F.Cu")
-		(at 146.3625 126.175)
+		(at 144.75 126.25)
 		(descr "Resistor SMD 0402 (1005 Metric), square (rectangular) end terminal, IPC-7351 nominal, (Body size source: IPC-SM-782 page 72, https://www.pcb-3d.com/wordpress/wp-content/uploads/ipc-sm-782a_amendment_1_and_2.pdf)")
 		(tags "resistor")
@@
 	)
 	(segment
-		(start 145.8425 124.925)
-		(end 144.825 124.925)
-		(width 0.2)
-		(layer "F.Cu")
-		(net "GND")
-	)
-	(segment
 		(start 141.5 129.27)
 		(end 140.5 129.27)
@@
 	)
 	(segment
-		(start 144.825 124.925)
-		(end 144.75 125)
+		(start 144.25 124)
+		(end 144.25 124.98)
 		(width 0.2)
 		(layer "F.Cu")
@@
 	)
 	(segment
+		(start 144.25 124.98)
+		(end 144.23 125)
+		(width 0.2)
+		(layer "F.Cu")
+		(net "GND")
+	)
+	(segment
 		(start 159.64 125.175)
 		(end 159.645 125.18)
@@
 	)
 	(via
-		(at 144.75 125)
+		(at 144.25 124)
 		(size 0.6)
 		(drill 0.3)
@@
 	)
 	(segment
-		(start 146.8725 126.175)
-		(end 146.8725 124.935)
+		(start 145.26 126.25)
+		(end 145.26 125.01)
 		(width 0.3)
 		(layer "F.Cu")
@@
 	)
 	(segment
-		(start 146.8725 124.935)
-		(end 146.8625 124.925)
+		(start 145.26 125.01)
+		(end 145.25 125)
 		(width 0.3)
 		(layer "F.Cu")

Commit message: Autosave
Routing:
- net /BOOT: track 0.00 -> 1.37 mm
- net Net-(R1-Pad2): track 8.02 -> 7.43 mm
Changed lines of the file:
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@@
 	)
 	(segment
-		(start 146.8625 124.02151)
-		(end 146.8625 124.925)
+		(start 145.25 122.40901)
+		(end 145.25 125)
 		(width 0.5)
 		(layer "F.Cu")
@@
 	(segment
 		(start 143.84099 121)
-		(end 146.8625 124.02151)
+		(end 145.25 122.40901)
 		(width 0.5)
 		(layer "F.Cu")
@@
 	)
 	(segment
+		(start 144.24 127.4725)
+		(end 144.1375 127.575)
+		(width 0.3)
+		(layer "F.Cu")
+		(net "/BOOT")
+	)
+	(segment
+		(start 144.24 126.25)
+		(end 144.24 127.4725)
+		(width 0.3)
+		(layer "F.Cu")
+		(net "/BOOT")
+	)
+	(segment

Commit message: Autosave
Parts:
- moved U1 0.25 mm to (147.0, 130.2)
Routing:
- net +3.3V: track 2.34 -> 21.1 mm
Changed lines of the file:
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@@
 	(footprint "Package_SO:TSSOP-20_4.4x6.5mm_P0.65mm"
 		(layer "F.Cu")
-		(at 147 130.5)
+		(at 147 130.25)
 		(descr "TSSOP, 20 Pin (JEDEC MO-153 Var AC https://www.jedec.org/document_search?search_api_views_fulltext=MO-153)")
 		(tags "TSSOP SO")
@@
 	)
 	(segment
+		(start 147.175 119.425)
+		(end 148.75 121)
+		(width 0.5)
+		(layer "F.Cu")
+		(net "+3.3V")
+	)
+	(segment
+		(start 142.02 125.25)
+		(end 142.02 122.997387)
+		(width 0.5)
+		(layer "F.Cu")
+		(net "+3.3V")
+	)
+	(segment
 		(start 137.25 124.25)
 		(end 137.75 124.25)
 		(width 0.3)
+		(layer "F.Cu")
+		(net "+3.3V")
+	)
+	(segment
+		(start 142.02 122.997387)
+		(end 140.675 121.652387)
+		(width 0.5)
+		(layer "F.Cu")
+		(net "+3.3V")
+	)
+	(segment
+		(start 140.675 120.347613)
+		(end 141.597613 119.425)
+		(width 0.5)
+		(layer "F.Cu")
+		(net "+3.3V")
+	)
+	(segment
+		(start 139.2875 125.075)
+		(end 140.8875 126.675)
+		(width 0.3)
+		(layer "F.Cu")
+		(net "+3.3V")
+	)
+	(segment
+		(start 140.675 121.652387)
+		(end 140.675 120.347613)
+		(width 0.5)
+		(layer "F.Cu")
+		(net "+3.3V")
+	)
+	(segment
+		(start 142.02 125.5425)
+		(end 140.8875 126.675)
+		(width 0.5)
+		(layer "F.Cu")
+		(net "+3.3V")
+	)
+	(segment
+		(start 141.597613 119.425)
+		(end 147.175 119.425)
+		(width 0.5)
 		(layer "F.Cu")
 		(net "+3.3V")
@@
 		(width 0.3)
 		(layer "F.Cu")
+		(net "+3.3V")
+	)
+	(segment
+		(start 142.02 125.25)
+		(end 142.02 125.5425)
+		(width 0.5)
+		(layer "F.Cu")
+		(net "+3.3V")
+	)
+	(segment
+		(start 139.25 125.075)
+		(end 139.2875 125.075)
+		(width 0.3)
+		(layer "F.Cu")

Commit message: Autosave
Parts:
- moved R1 0.25 mm to (144.7, 124.8)
- moved R6 0.25 mm to (144.8, 126.0)
Changed lines of the file:
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@@
 	(footprint "Resistor_SMD:R_0402_1005Metric"
 		(layer "F.Cu")
-		(at 144.74 125)
+		(at 144.74 124.75)
 		(descr "Resistor SMD 0402 (1005 Metric), square (rectangular) end terminal, IPC-7351 nominal, (Body size source: IPC-SM-782 page 72, https://www.pcb-3d.com/wordpress/wp-content/uploads/ipc-sm-782a_amendment_1_and_2.pdf)")
 		(tags "resistor")
@@
 	(footprint "Resistor_SMD:R_0402_1005Metric"
 		(layer "F.Cu")
-		(at 144.75 126.25)
+		(at 144.75 126)
 		(descr "Resistor SMD 0402 (1005 Metric), square (rectangular) end terminal, IPC-7351 nominal, (Body size source: IPC-SM-782 page 72, https://www.pcb-3d.com/wordpress/wp-content/uploads/ipc-sm-782a_amendment_1_and_2.pdf)")
 		(tags "resistor")
@@
 	)
 	(via
-		(at 144.25 124)
+		(at 144.25 123.75)
 		(size 0.6)
 		(drill 0.3)
@@
 	)
 	(segment
-		(start 144.24 127.4725)
-		(end 144.1375 127.575)
+		(start 144.24 127.2225)
+		(end 144.1375 127.325)
 		(width 0.3)
 		(layer "F.Cu")
@@
 	(segment
 		(start 144.24 126.25)
-		(end 144.24 127.4725)
+		(end 144.24 127.2225)
 		(width 0.3)
 		(layer "F.Cu")

Commit message: Autosave
Routing:
- net RECV_PWM: track 11.2 -> 17.2 mm
Changed lines of the file:
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@@
+	)
+	(segment
+		(start 138.325 131.075)
+		(end 142.661846 131.075)
+		(width 0.3)
+		(layer "F.Cu")
+		(net "RECV_PWM")
+	)
+	(segment
+		(start 142.661846 131.075)
+		(end 143.161846 130.575)
+		(width 0.3)
+		(layer "F.Cu")
+		(net "RECV_PWM")
 	)
 	(segment
@@
 		(layer "F.Cu")
 		(net "RECV_PWM")
+	)
+	(segment
+		(start 143.161846 130.575)
+		(end 144.1375 130.575)
+		(width 0.3)
+		(layer "F.Cu")
+		(net "RECV_PWM")

Commit message: Autosave
Parts:
- moved R4 0.25 mm to (142.2, 132.5)
Changed lines of the file:
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@@
 	(footprint "Resistor_SMD:R_0402_1005Metric"
 		(layer "F.Cu")
-		(at 142.5 132.5 90)
+		(at 142.25 132.5 90)
 		(descr "Resistor SMD 0402 (1005 Metric), square (rectangular) end terminal, IPC-7351 nominal, (Body size source: IPC-SM-782 page 72, https://www.pcb-3d.com/wordpress/wp-content/uploads/ipc-sm-782a_amendment_1_and_2.pdf)")
 		(tags "resistor")

Commit message: Autosave
Parts:
- moved C3 0.25 mm to (140.5, 129.5)
- moved C4 0.25 mm to (141.5, 129.5)
- moved C6 0.25 mm to (142.5, 129.5)
Routing:
- net /NRST: track 0.00 -> 1.74 mm
- net GND: track 17.7 -> 16.7 mm
Changed lines of the file:
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@@
 	(footprint "Capacitor_SMD:C_0402_1005Metric"
 		(layer "F.Cu")
-		(at 142.5 129.75 -90)
+		(at 142.5 129.5 -90)
 		(descr "Capacitor SMD 0402 (1005 Metric), square (rectangular) end terminal, IPC-7351 nominal, (Body size source: IPC-SM-782 page 76, https://www.pcb-3d.com/wordpress/wp-content/uploads/ipc-sm-782a_amendment_1_and_2.pdf)")
 		(tags "capacitor")
@@
 	(footprint "Capacitor_SMD:C_0402_1005Metric"
 		(layer "F.Cu")
-		(at 141.5 129.75 90)
+		(at 141.5 129.5 90)
 		(descr "Capacitor SMD 0402 (1005 Metric), square (rectangular) end terminal, IPC-7351 nominal, (Body size source: IPC-SM-782 page 76, https://www.pcb-3d.com/wordpress/wp-content/uploads/ipc-sm-782a_amendment_1_and_2.pdf)")
 		(tags "capacitor")
@@
 	(footprint "Capacitor_SMD:C_0402_1005Metric"
 		(layer "F.Cu")
-		(at 140.5 129.75 90)
+		(at 140.5 129.5 90)
 		(descr "Capacitor SMD 0402 (1005 Metric), square (rectangular) end terminal, IPC-7351 nominal, (Body size source: IPC-SM-782 page 76, https://www.pcb-3d.com/wordpress/wp-content/uploads/ipc-sm-782a_amendment_1_and_2.pdf)")
 		(tags "capacitor")
@@
 	)
 	(segment
-		(start 141.5 129.27)
-		(end 140.5 129.27)
-		(width 0.3)
-		(layer "F.Cu")
-		(net "GND")
-	)
-	(segment
 		(start 159.07 126.3)
 		(end 159.07 125.755)
@@
 	)
 	(segment
+		(start 142.5 129.02)
+		(end 142.755 129.275)
+		(width 0.3)
+		(layer "F.Cu")
+		(net "/NRST")
+	)
+	(segment
+		(start 142.755 129.275)
+		(end 144.1375 129.275)
+		(width 0.3)
+		(layer "F.Cu")
+		(net "/NRST")
+	)
+	(segment

Commit message: Autosave
Routing:
- net GND: track 16.7 -> 17.7 mm
Changed lines of the file:
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@@
+	)
+	(segment
+		(start 140.5 129.02)
+		(end 141.5 129.02)
+		(width 0.3)
+		(layer "F.Cu")
+		(net "GND")
 	)
 	(segment
