File: AeroBlinker.kicad_pcb (KiCad board)
At the start: 2 copper layers, 41.8 x 28 mm, 33 parts, among them J1 LED_GND, J2 LED_GND, J3 LED_GND, J4 BATTERY, J5 RECEIVER, J6 USB_C_Receptacle_USB2.0_16P, Q1 AO3400A, SW2 SW_Push, U1 STM32F042F6Px, U2 USBLC6-2SC6, U3 TPS62162DGR

Commit message: Autosave
Routing:
- net /USB_D+: track 5.13 -> 7.84 mm
Changed lines of the file:
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@@
 	)
 	(segment
-		(start 152.076 127.861)
-		(end 152.076 128.389)
+		(start 152.3225 128.625)
+		(end 153.1875 128.625)
 		(width 0.3)
 		(layer "F.Cu")
@@
 	)
 	(segment
-		(start 151.486 128.389)
-		(end 151.486 127.861)
-		(width 0.3)
-		(layer "F.Cu")
-		(net "/USB_D+")
-	)
-	(segment
-		(start 152.312 128.625)
-		(end 152.43 128.625)
+		(start 151.9685 126.507204)
+		(end 151.9685 128.389)
 		(width 0.3)
 		(layer "F.Cu")
@@
 	(segment
 		(start 149.8625 128.625)
-		(end 151.25 128.625)
-		(width 0.3)
-		(layer "F.Cu")
-		(net "/USB_D+")
-	)
-	(segment
-		(start 151.722 127.625)
-		(end 151.84 127.625)
+		(end 150.5025 128.625)
 		(width 0.3)
 		(layer "F.Cu")
@@
 	)
 	(segment
-		(start 152.872899 128.625)
-		(end 153.1875 128.625)
+		(start 152.2045 128.625)
+		(end 152.3225 128.625)
 		(width 0.3)
 		(layer "F.Cu")
@@
 	)
 	(segment
-		(start 152.43 128.625)
-		(end 152.872899 128.625)
+		(start 150.5025 128.625)
+		(end 151.1425 128.625)
+		(width 0.3)
+		(layer "F.Cu")
+		(net "/USB_D+")
+	)
+	(segment
+		(start 151.6145 126.271204)
+		(end 151.7325 126.271204)
+		(width 0.3)
+		(layer "F.Cu")
+		(net "/USB_D+")
+	)
+	(segment
+		(start 151.3785 128.389)
+		(end 151.3785 126.507204)
 		(width 0.3)
 		(layer "F.Cu")
@@
 	)
 	(arc
-		(start 151.25 128.625)
-		(mid 151.416877 128.555877)
-		(end 151.486 128.389)
+		(start 151.3785 126.507204)
+		(mid 151.447623 126.340327)
+		(end 151.6145 126.271204)
 		(width 0.3)
 		(layer "F.Cu")
@@
 	)
 	(arc
-		(start 151.486 127.861)
-		(mid 151.555123 127.694123)
-		(end 151.722 127.625)
+		(start 151.7325 126.271204)
+		(mid 151.899377 126.340327)
+		(end 151.9685 126.507204)
 		(width 0.3)
 		(layer "F.Cu")
@@
 	)
 	(arc
-		(start 151.84 127.625)
-		(mid 152.006877 127.694123)
-		(end 152.076 127.861)
+		(start 151.9685 128.389)
+		(mid 152.037623 128.555877)
+		(end 152.2045 128.625)
 		(width 0.3)
 		(layer "F.Cu")
@@
 	)
 	(arc
-		(start 152.076 128.389)
-		(mid 152.145123 128.555877)
-		(end 152.312 128.625)
+		(start 151.1425 128.625)
+		(mid 151.309377 128.555877)
+		(end 151.3785 128.389)
 		(width 0.3)
 		(layer "F.Cu")
@@
 		(base_line
 			(pts
-				(xy 151.25 128.625) (xy 152.872899 128.625)
+				(xy 149.8625 128.625) (xy 153.1875 128.625) (xy 153.3625 128.45)
 			)
 		)
@@
 		(corner_radius_percent 80)
 		(end
-			(xy 152.872899 128.625)
+			(xy 153.3625 128.45)
 		)
 		(initial_side "left")
@@
 		(last_diff_pair_gap 0.18)
 		(last_netname "/USB_D+")
-		(last_status "too_short")
+		(last_status "tuned")
 		(last_track_width 0.3)
-		(last_tuning_length -2.707586)
-		(max_amplitude 1)
+		(last_tuning_length 8e-06)
+		(max_amplitude 3.41)
 		(min_amplitude 0.2)
 		(min_spacing 0.59)
 		(origin
-			(xy 151.25 128.625)
+			(xy 149.8625 128.625)
 		)
 		(override_custom_rules no)
@@
 		(target_skew_min -0.1)
 		(tuning_mode "diff_pair_skew")
-		(members "0d66e9a5-57ea-49d4-afdd-e1d03e306a11" "2244ac87-f69b-496b-b926-40137be1e190"
-			"4f72bb4b-5ca8-46af-b09f-82ce8b472de2" "5b351391-ae3a-42b1-babb-cb6b179e0d81"
-			"77059792-058e-4a97-a2d5-626a9b3ab519" "9b82336f-540b-47c4-b436-318d57764b23"
-			"aa575962-a515-4c9d-a1f2-eb061a80591c" "c143c16c-24e8-4597-b7bc-3079f5318614"
-			"fa6b5e54-2679-494e-a93d-aa4f8f90b363"
+		(members "0f98827f-2dbb-465a-b232-4244514e80dd" "26b30922-d3f1-485b-ad6f-2d03c6639e9a"
+			"37007184-a848-4b24-bd9d-d222cd75f9c9" "38f7b7d8-e85c-4034-a57c-b45d56f05c9a"
+			"3cd1f93c-8f1b-4630-a3ef-e4ad4eb656eb" "420af76d-2cb4-40ea-84db-06e455cc811a"
+			"6efca980-59e1-4a95-94c6-34c594cbb825" "725d132c-afa0-4fc2-8e9b-75623586d88d"
+			"753f3dee-1099-4363-9c97-457d54d11d85" "84d0f110-b759-498c-bf18-f2befbb7b15b"
+			"95401eb1-143a-4136-9788-26018892537c" "b13fd1ba-43d2-4499-801e-21ac679f2428"
 		)
 	)

Commit message: Autosave
Parts:
- turned U2 to 90 degrees
Changed lines of the file:
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@@
 	(footprint "Package_TO_SOT_SMD:SOT-23-6"
 		(layer "F.Cu")
-		(at 154.5 127.5 180)
+		(at 154.5 127.5 90)
 		(descr "SOT, 6 Pin (JEDEC MO-178 Var AB https://www.jedec.org/document_search?search_api_views_fulltext=MO-178)")
 		(tags "SOT TO_SOT_SMD")
 		(property "Reference" "U2"
-			(at 3 -0.075 0)
+			(at 3 -0.075 90)
 			(layer "F.SilkS")
 			(effects
@@
 		)
 		(property "Value" "USBLC6-2SC6"
-			(at 0 2.4 0)
+			(at 0 2.4 90)
 			(layer "F.Fab")
 			(effects
@@
 		)
 		(property "Datasheet" "https://www.st.com/resource/en/datasheet/usblc6-2.pdf"
-			(at 0 0 0)
+			(at 0 0 90)
 			(layer "F.Fab")
 			(hide yes)
@@
 		)
 		(property "Description" "Very low capacitance ESD protection diode, 2 data-line, SOT-23-6"
-			(at 0 0 0)
+			(at 0 0 90)
 			(layer "F.Fab")
 			(hide yes)
@@
 		)
 		(property "KiLib_Generator" "package/gullwing"
-			(at 0 0 0)
+			(at 0 0 90)
 			(layer "F.SilkS")
 			(hide yes)
@@
 		(duplicate_pad_numbers_are_jumpers no)
 		(fp_line
+			(start 0.91 -1.56)
+			(end 0.91 -1.51)
+			(stroke
+				(width 0.12)
+				(type solid)
+			)
+			(layer "F.SilkS")
+		)
+		(fp_line
+			(start -0.91 -1.56)
+			(end 0.91 -1.56)
+			(stroke
+				(width 0.12)
+				(type solid)
+			)
+			(layer "F.SilkS")
+		)
+		(fp_line
+			(start -0.91 -1.51)
+			(end -0.91 -1.56)
+			(stroke
+				(width 0.12)
+				(type solid)
+			)
+			(layer "F.SilkS")
+		)
+		(fp_line
+			(start 0.91 1.51)
+			(end 0.91 1.56)
+			(stroke
+				(width 0.12)
+				(type solid)
+			)
+			(layer "F.SilkS")
+		)
+		(fp_line
 			(start 0.91 1.56)
 			(end -0.91 1.56)
@@
 		)
 		(fp_line
-			(start 0.91 1.51)
-			(end 0.91 1.56)
-			(stroke
-				(width 0.12)
-				(type solid)
-			)
-			(layer "F.SilkS")
-		)
-		(fp_line
-			(start 0.91 -1.56)
-			(end 0.91 -1.51)
-			(stroke
-				(width 0.12)
-				(type solid)
-			)
-			(layer "F.SilkS")
-		)
-		(fp_line
 			(start -0.91 1.56)
 			(end -0.91 1.51)
-			(stroke
-				(width 0.12)
-				(type solid)
-			)
-			(layer "F.SilkS")
-		)
-		(fp_line
-			(start -0.91 -1.51)
-			(end -0.91 -1.56)
-			(stroke
-				(width 0.12)
-				(type solid)
-			)
-			(layer "F.SilkS")
-		)
-		(fp_line
-			(start -0.91 -1.56)
-			(end 0.91 -1.56)
 			(stroke
 				(width 0.12)
@@
 		)
 		(fp_line
+			(start 1.05 -1.7)
+			(end 1.05 -1.5)
+			(stroke
+				(width 0.05)
+				(type solid)
+			)
+			(layer "F.CrtYd")
+		)
+		(fp_line
+			(start -1.05 -1.7)
+			(end 1.05 -1.7)
+			(stroke
+				(width 0.05)
+				(type solid)
+			)
+			(layer "F.CrtYd")
+		)
+		(fp_line
+			(start 2.05 -1.5)
+			(end 2.05 1.5)
+			(stroke
+				(width 0.05)
+				(type solid)
+			)
+			(layer "F.CrtYd")
+		)
+		(fp_line
+			(start 1.05 -1.5)
+			(end 2.05 -1.5)
+			(stroke
+				(width 0.05)
+				(type solid)
+			)
+			(layer "F.CrtYd")
+		)
+		(fp_line
+			(start -1.05 -1.5)
+			(end -1.05 -1.7)
+			(stroke
+				(width 0.05)
+				(type solid)
+			)
+			(layer "F.CrtYd")
+		)
+		(fp_line
+			(start -2.05 -1.5)
+			(end -1.05 -1.5)
+			(stroke
+				(width 0.05)
+				(type solid)
+			)
+			(layer "F.CrtYd")
+		)
+		(fp_line
 			(start 2.05 1.5)
 			(end 1.05 1.5)
@@
 		)
 		(fp_line
-			(start 2.05 -1.5)
-			(end 2.05 1.5)
+			(start 1.05 1.5)
+			(end 1.05 1.7)
+			(stroke
+				(width 0.05)
+				(type solid)
+			)
+			(layer "F.CrtYd")
+		)
+		(fp_line
+			(start -1.05 1.5)
+			(end -2.05 1.5)
+			(stroke
+				(width 0.05)
+				(type solid)
+			)
+			(layer "F.CrtYd")
+		)
+		(fp_line
+			(start -2.05 1.5)
+			(end -2.05 -1.5)
 			(stroke
 				(width 0.05)
@@
 		)
 		(fp_line
-			(start 1.05 1.5)
-			(end 1.05 1.7)
-			(stroke
-				(width 0.05)
-				(type solid)
-			)
-			(layer "F.CrtYd")
-		)
-		(fp_line
-			(start 1.05 -1.5)
-			(end 2.05 -1.5)
-			(stroke
-				(width 0.05)
-				(type solid)
-			)
-			(layer "F.CrtYd")
-		)
-		(fp_line
-			(start 1.05 -1.7)
-			(end 1.05 -1.5)
-			(stroke
-				(width 0.05)
-				(type solid)
-			)
-			(layer "F.CrtYd")
-		)
-		(fp_line
 			(start -1.05 1.7)
 			(end -1.05 1.5)
-			(stroke
-				(width 0.05)
-				(type solid)
-			)
-			(layer "F.CrtYd")
-		)
-		(fp_line
-			(start -1.05 1.5)
-			(end -2.05 1.5)
-			(stroke
-				(width 0.05)
-				(type solid)
-			)
-			(layer "F.CrtYd")
-		)
-		(fp_line
-			(start -1.05 -1.5)
-			(end -1.05 -1.7)
-			(stroke
-				(width 0.05)
-				(type solid)
-			)
-			(layer "F.CrtYd")
-		)
-		(fp_line
-			(start -1.05 -1.7)
-			(end 1.05 -1.7)
-			(stroke
-				(width 0.05)
-				(type solid)
-			)
-			(layer "F.CrtYd")
-		)
-		(fp_line
-			(start -2.05 1.5)
-			(end -2.05 -1.5)
-			(stroke
-				(width 0.05)
-				(type solid)
-			)
-			(layer "F.CrtYd")
-		)
-		(fp_line
-			(start -2.05 -1.5)
-			(end -1.05 -1.5)
 			(stroke
 				(width 0.05)
@@
 		)
 		(fp_text user "${REFERENCE}"
-			(at 0 0 90)
+			(at 0 0 0)
 			(layer "F.Fab")
 			(effects
@@
 		)
 		(pad "1" smd roundrect
-			(at -1.1375 -0.95 180)
+			(at -1.1375 -0.95 90)
 			(size 1.325 0.6)
 			(layers "F.Cu" "F.Mask" "F.Paste")
@@
 		)
 		(pad "2" smd roundrect
-			(at -1.1375 0 180)
+			(at -1.1375 0 90)
 			(size 1.325 0.6)
 			(layers "F.Cu" "F.Mask" "F.Paste")
@@
 		)
 		(pad "3" smd roundrect
-			(at -1.1375 0.95 180)
+			(at -1.1375 0.95 90)
 			(size 1.325 0.6)
 			(layers "F.Cu" "F.Mask" "F.Paste")
@@
 		)
 		(pad "4" smd roundrect
-			(at 1.1375 0.95 180)
+			(at 1.1375 0.95 90)
 			(size 1.325 0.6)
 			(layers "F.Cu" "F.Mask" "F.Paste")
@@
 		)
 		(pad "5" smd roundrect
-			(at 1.1375 0 180)
+			(at 1.1375 0 90)
 			(size 1.325 0.6)
 			(layers "F.Cu" "F.Mask" "F.Paste")
@@
 		)
 		(pad "6" smd roundrect
-			(at 1.1375 -0.95 180)
-			(size 1.325 0.6)
-			(layers "F.Cu" "F.Mask" "F.Paste")
+			(at 1.1375 -0.95 90)
+			(size 1.325 0.6)
+			(layers "F.Cu" "F.Mask" "F.Paste")

Commit message: Autosave
Routing:
- net /USB_D+: track 7.84 -> 0.00 mm
Changed lines of the file:
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@@
 		(net "/USB_D-")
-	)
-	(segment
-		(start 152.3225 128.625)
-		(end 153.1875 128.625)
-		(width 0.3)
-		(layer "F.Cu")
-		(net "/USB_D+")
-	)
-	(segment
-		(start 151.9685 126.507204)
-		(end 151.9685 128.389)
-		(width 0.3)
-		(layer "F.Cu")
-		(net "/USB_D+")
-	)
-	(segment
-		(start 149.8625 128.625)
-		(end 150.5025 128.625)
-		(width 0.3)
-		(layer "F.Cu")
-		(net "/USB_D+")
-	)
-	(segment
-		(start 153.1875 128.625)
-		(end 153.3625 128.45)
-		(width 0.3)
-		(layer "F.Cu")
-		(net "/USB_D+")
-	)
-	(segment
-		(start 152.2045 128.625)
-		(end 152.3225 128.625)
-		(width 0.3)
-		(layer "F.Cu")
-		(net "/USB_D+")
-	)
-	(segment
-		(start 150.5025 128.625)
-		(end 151.1425 128.625)
-		(width 0.3)
-		(layer "F.Cu")
-		(net "/USB_D+")
-	)
-	(segment
-		(start 151.6145 126.271204)
-		(end 151.7325 126.271204)
-		(width 0.3)
-		(layer "F.Cu")
-		(net "/USB_D+")
-	)
-	(segment
-		(start 151.3785 128.389)
-		(end 151.3785 126.507204)
-		(width 0.3)
-		(layer "F.Cu")
-		(net "/USB_D+")
-	)
-	(arc
-		(start 151.3785 126.507204)
-		(mid 151.447623 126.340327)
-		(end 151.6145 126.271204)
-		(width 0.3)
-		(layer "F.Cu")
-		(net "/USB_D+")
-	)
-	(arc
-		(start 151.7325 126.271204)
-		(mid 151.899377 126.340327)
-		(end 151.9685 126.507204)
-		(width 0.3)
-		(layer "F.Cu")
-		(net "/USB_D+")
-	)
-	(arc
-		(start 151.9685 128.389)
-		(mid 152.037623 128.555877)
-		(end 152.2045 128.625)
-		(width 0.3)
-		(layer "F.Cu")
-		(net "/USB_D+")
-	)
-	(arc
-		(start 151.1425 128.625)
-		(mid 151.309377 128.555877)
-		(end 151.3785 128.389)
-		(width 0.3)
-		(layer "F.Cu")
-		(net "/USB_D+")
 	)
 	(zone
@@
 		)
 	)
-	(generated
-		(type tuning_pattern)
-		(name "Tuning Pattern")
-		(layer "F.Cu")
-		(base_line
-			(pts
-				(xy 149.8625 128.625) (xy 153.1875 128.625) (xy 153.3625 128.45)
-			)
-		)
-		(base_line_coupled
-			(pts
-				(xy 151.561064 129.275) (xy 151.56759 129.275)
-			)
-		)
-		(corner_radius_percent 80)
-		(end
-			(xy 153.3625 128.45)
-		)
-		(initial_side "left")
-		(is_time_domain no)
-		(last_diff_pair_gap 0.18)
-		(last_netname "/USB_D+")
-		(last_status "tuned")
-		(last_track_width 0.3)
-		(last_tuning_length 8e-06)
-		(max_amplitude 3.41)
-		(min_amplitude 0.2)
-		(min_spacing 0.59)
-		(origin
-			(xy 149.8625 128.625)
-		)
-		(override_custom_rules no)
-		(rounded yes)
-		(single_sided no)
-		(target_delay 1000000)
-		(target_delay_max 1000000)
-		(target_delay_min 0)
-		(target_length 1000000)
-		(target_length_max 1000000)
-		(target_length_min 0)
-		(target_skew 0)
-		(target_skew_max 0.1)
-		(target_skew_min -0.1)
-		(tuning_mode "diff_pair_skew")
-		(members "0f98827f-2dbb-465a-b232-4244514e80dd" "26b30922-d3f1-485b-ad6f-2d03c6639e9a"
-			"37007184-a848-4b24-bd9d-d222cd75f9c9" "38f7b7d8-e85c-4034-a57c-b45d56f05c9a"
-			"3cd1f93c-8f1b-4630-a3ef-e4ad4eb656eb" "420af76d-2cb4-40ea-84db-06e455cc811a"
-			"6efca980-59e1-4a95-94c6-34c594cbb825" "725d132c-afa0-4fc2-8e9b-75623586d88d"
-			"753f3dee-1099-4363-9c97-457d54d11d85" "84d0f110-b759-498c-bf18-f2befbb7b15b"
-			"95401eb1-143a-4136-9788-26018892537c" "b13fd1ba-43d2-4499-801e-21ac679f2428"
-		)
-	)

Commit message: Autosave
Parts:
- moved C2 0.50 mm to (153.0, 131.8)
Routing:
- net /USB_D+: track 0.00 -> 4.62 mm
- net /USB_D-: track 7.83 -> 7.05 mm
Changed lines of the file:
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@@
 	(footprint "Capacitor_SMD:C_0603_1608Metric"
 		(layer "F.Cu")
-		(at 153 131.25 -90)
+		(at 153 131.75 -90)
 		(descr "Capacitor SMD 0603 (1608 Metric), square (rectangular) end terminal, IPC-7351 nominal, (Body size source: IPC-SM-782 page 76, https://www.pcb-3d.com/wordpress/wp-content/uploads/ipc-sm-782a_amendment_1_and_2.pdf)")
 		(tags "capacitor")
@@
 	)
 	(segment
-		(start 153.975 129.275)
-		(end 154.375 128.875)
+		(start 149.8625 129.275)
+		(end 151.475 129.275)
 		(width 0.3)
 		(layer "F.Cu")
@@
 	)
 	(segment
-		(start 154.375 128.875)
-		(end 154.375 126.875)
+		(start 155.45 126.8)
+		(end 155.45 126.3625)
 		(width 0.3)
 		(layer "F.Cu")
@@
 	)
 	(segment
-		(start 154.05 126.55)
-		(end 153.3625 126.55)
+		(start 151.475 129.275)
+		(end 153.375 127.375)
 		(width 0.3)
 		(layer "F.Cu")
@@
 	)
 	(segment
-		(start 154.375 126.875)
-		(end 154.05 126.55)
+		(start 154.875 127.375)
+		(end 155.45 126.8)
 		(width 0.3)
 		(layer "F.Cu")
@@
 	)
 	(segment
-		(start 149.8625 129.275)
-		(end 153.975 129.275)
+		(start 153.375 127.375)
+		(end 154.875 127.375)
 		(width 0.3)
 		(layer "F.Cu")
 		(net "/USB_D-")
 	)
+	(segment
+		(start 151.2875 128.625)
+		(end 153.55 126.3625)
+		(width 0.3)
+		(layer "F.Cu")
+		(net "/USB_D+")
+	)
+	(segment
+		(start 149.8625 128.625)
+		(end 151.2875 128.625)
+		(width 0.3)
+		(layer "F.Cu")
+		(net "/USB_D+")
+	)
 	(zone

Commit message: Autosave
Parts:
- moved C2 0.25 mm to (152.8, 131.8)
Routing:
- net /USB_D-: track 7.05 -> 0.00 mm
Changed lines of the file:
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@@
 	(footprint "Capacitor_SMD:C_0603_1608Metric"
 		(layer "F.Cu")
-		(at 153 131.75 -90)
+		(at 152.75 131.75 -90)
 		(descr "Capacitor SMD 0603 (1608 Metric), square (rectangular) end terminal, IPC-7351 nominal, (Body size source: IPC-SM-782 page 76, https://www.pcb-3d.com/wordpress/wp-content/uploads/ipc-sm-782a_amendment_1_and_2.pdf)")
 		(tags "capacitor")
@@
 	)
 	(segment
-		(start 149.8625 129.275)
-		(end 151.475 129.275)
-		(width 0.3)
-		(layer "F.Cu")
-		(net "/USB_D-")
-	)
-	(segment
-		(start 155.45 126.8)
-		(end 155.45 126.3625)
-		(width 0.3)
-		(layer "F.Cu")
-		(net "/USB_D-")
-	)
-	(segment
-		(start 151.475 129.275)
-		(end 153.375 127.375)
-		(width 0.3)
-		(layer "F.Cu")
-		(net "/USB_D-")
-	)
-	(segment
-		(start 154.875 127.375)
-		(end 155.45 126.8)
-		(width 0.3)
-		(layer "F.Cu")
-		(net "/USB_D-")
-	)
-	(segment
-		(start 153.375 127.375)
-		(end 154.875 127.375)
-		(width 0.3)
-		(layer "F.Cu")
-		(net "/USB_D-")
-	)
-	(segment

Commit message: Autosave
Parts:
- moved U2 2.14 mm to (155.2, 129.5)
Routing:
- net /USB_D+: track 4.62 -> 0.00 mm
Changed lines of the file:
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@@
 	(footprint "Package_TO_SOT_SMD:SOT-23-6"
 		(layer "F.Cu")
-		(at 154.5 127.5 90)
+		(at 155.25 129.5 90)
 		(descr "SOT, 6 Pin (JEDEC MO-178 Var AB https://www.jedec.org/document_search?search_api_views_fulltext=MO-178)")
 		(tags "SOT TO_SOT_SMD")
@@
 		(net "/LED_GATE")
 	)
-	(segment
-		(start 151.2875 128.625)
-		(end 153.55 126.3625)
-		(width 0.3)
-		(layer "F.Cu")
-		(net "/USB_D+")
-	)
-	(segment
-		(start 149.8625 128.625)
-		(end 151.2875 128.625)
-		(width 0.3)
-		(layer "F.Cu")
-		(net "/USB_D+")
-	)
 	(zone

Commit message: Autosave
Routing:
- net Net-(J6-D--PadA7): track 0.00 -> 5.73 mm
- net Net-(J6-D+-PadA6): track 0.00 -> 3.24 mm
Changed lines of the file:
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@@
 		(net "/LED_GATE")
+	)
+	(segment
+		(start 156.880394 129.25)
+		(end 159.07 129.25)
+		(width 0.3)
+		(layer "F.Cu")
+		(net "Net-(J6-D--PadA7)")
+	)
+	(segment
+		(start 154.3 130.6375)
+		(end 154.3 129.975001)
+		(width 0.3)
+		(layer "F.Cu")
+		(net "Net-(J6-D--PadA7)")
+	)
+	(segment
+		(start 156.690196 129.440197)
+		(end 156.880394 129.25)
+		(width 0.3)
+		(layer "F.Cu")
+		(net "Net-(J6-D--PadA7)")
+	)
+	(segment
+		(start 154.3 129.975001)
+		(end 154.834804 129.440197)
+		(width 0.3)
+		(layer "F.Cu")
+		(net "Net-(J6-D--PadA7)")
+	)
+	(segment
+		(start 154.834804 129.440197)
+		(end 156.690196 129.440197)
+		(width 0.3)
+		(layer "F.Cu")
+		(net "Net-(J6-D--PadA7)")
+	)
+	(segment
+		(start 156.2 130.6375)
+		(end 157.0875 129.75)
+		(width 0.3)
+		(layer "F.Cu")
+		(net "Net-(J6-D+-PadA6)")
+	)
+	(segment
+		(start 157.0875 129.75)
+		(end 159.07 129.75)
+		(width 0.3)
+		(layer "F.Cu")
+		(net "Net-(J6-D+-PadA6)")
 	)
 	(zone

Commit message: Autosave
Parts:
- added TP2: TestPoint, TestPoint:TestPoint_2Pads_Pitch5.08mm_Drill1.3mm, F.Cu at (1.82, 1.82)
- R3: footprint Resistor_SMD:R_0402_1005Metric -> Resistor_SMD:R_0603_1608Metric
Connections:
- TP1 pad 1: /SYS_SWDIO -> /SYS_SWCLK
- TP1 pad 2: /SYS_SWCLK -> (no net)
Changed lines of the file:
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@@
 		(embedded_fonts no)
 	)
-	(footprint "Resistor_SMD:R_0402_1005Metric"
+	(footprint "Resistor_SMD:R_0603_1608Metric"
 		(layer "F.Cu")
 		(at 157.25 127 90)
-		(descr "Resistor SMD 0402 (1005 Metric), square (rectangular) end terminal, IPC-7351 nominal, (Body size source: IPC-SM-782 page 72, https://www.pcb-3d.com/wordpress/wp-content/uploads/ipc-sm-782a_amendment_1_and_2.pdf)")
+		(descr "Resistor SMD 0603 (1608 Metric), square (rectangular) end terminal, IPC-7351 nominal, (Body size source: IPC-SM-782 page 72, https://www.pcb-3d.com/wordpress/wp-content/uploads/ipc-sm-782a_amendment_1_and_2.pdf)")
 		(tags "resistor")
 		(property "Reference" "R3"
-			(at 1.75 -0.25 180)
+			(at 0 -1.43 90)
 			(layer "F.SilkS")
 			(effects
@@
 		)
 		(property "Value" "5K"
-			(at 0 1.17 90)
+			(at 0 1.43 90)
 			(layer "F.Fab")
 			(effects
@@
 		(duplicate_pad_numbers_are_jumpers no)
 		(fp_line
-			(start -0.153641 -0.38)
-			(end 0.153641 -0.38)
-			(stroke
-				(width 0.12)
-				(type solid)
-			)
-			(layer "F.SilkS")
-		)
-		(fp_line
-			(start -0.153641 0.38)
-			(end 0.153641 0.38)
+			(start -0.237258 -0.5225)
+			(end 0.237258 -0.5225)
+			(stroke
+				(width 0.12)
+				(type solid)
+			)
+			(layer "F.SilkS")
+		)
+		(fp_line
+			(start -0.237258 0.5225)
+			(end 0.237258 0.5225)
 			(stroke
 				(width 0.12)
@@
 		)
 		(fp_rect
-			(start -0.93 -0.47)
-			(end 0.93 0.47)
+			(start -1.48 -0.73)
+			(end 1.48 0.73)
 			(stroke
 				(width 0.05)
@@
 		)
 		(fp_rect
-			(start -0.525 -0.27)
-			(end 0.525 0.27)
+			(start -0.8 -0.4125)
+			(end 0.8 0.4125)
 			(stroke
 				(width 0.1)
@@
 			(effects
 				(font
-					(size 0.26 0.26)
-					(thickness 0.04)
+					(size 0.4 0.4)
+					(thickness 0.06)
 				)
 			)
 		)
 		(pad "1" smd roundrect
-			(at -0.51 0 90)
-			(size 0.54 0.64)
+			(at -0.825 0 90)
+			(size 0.8 0.95)
 			(layers "F.Cu" "F.Mask" "F.Paste")
 			(roundrect_rratio 0.25)
@@
 		)
 		(pad "2" smd roundrect
-			(at 0.51 0 90)
-			(size 0.54 0.64)
+			(at 0.825 0 90)
+			(size 0.8 0.95)
 			(layers "F.Cu" "F.Mask" "F.Paste")
 			(roundrect_rratio 0.25)
@@
 		)
 		(embedded_fonts no)
-		(model "${KICAD10_3DMODEL_DIR}/Resistor_SMD.3dshapes/R_0402_1005Metric.step"
+		(model "${KICAD10_3DMODEL_DIR}/Resistor_SMD.3dshapes/R_0603_1608Metric.step"
 			(offset
 				(xyz 0 0 0)
@@
 			)
 		)
+	)
+	(footprint "TestPoint:TestPoint_2Pads_Pitch5.08mm_Drill1.3mm"
+		(layer "F.Cu")
+		(at 1.825 1.825)
+		(descr "Test point with 2 pads, pitch 5.08mm, hole diameter 1.3mm, wire diameter 1.0mm")
+		(tags "CONN DEV")
+		(property "Reference" "TP2"
+			(at 2.54 -2.5 0)
+			(layer "F.SilkS")
+			(effects
+				(font
+					(size 1 1)
+					(thickness 0.15)
+				)
+			)
+		)
+		(property "Value" "TestPoint"
+			(at 2.54 3 0)
+			(layer "F.Fab")
+			(effects
+				(font
+					(size 1 1)
+					(thickness 0.15)
+				)
+			)
+		)
+		(property "Datasheet" ""
+			(at 0 0 0)
+			(unlocked yes)
+			(layer "F.Fab")
+			(hide yes)
+			(effects
+				(font
+					(size 1.27 1.27)
+					(thickness 0.15)
+				)
+			)
+		)
+		(property "Description" "test point"
+			(at 0 0 0)
+			(unlocked yes)
+			(layer "F.Fab")
+			(hide yes)
+			(effects
+				(font
+					(size 1.27 1.27)
+					(thickness 0.15)
+				)
+			)
+		)
+		(property ki_fp_filters "Pin* Test*")
+		(sheetname "/")
+		(sheetfile "AeroBlinker.kicad_sch")
+		(units
+			(unit
+				(name "A")
+				(pins "1")
+			)
+		)
+		(duplicate_pad_numbers_are_jumpers no)
+		(fp_line
+			(start -1.5 -1.5)
+			(end -1.5 1.5)
+			(stroke
+				(width 0.12)
+				(type solid)
+			)
+			(layer "F.SilkS")
+		)
+		(fp_line
+			(start -1.5 -1.5)
+			(end 6.6 -1.5)
+			(stroke
+				(width 0.12)
+				(type solid)
+			)
+			(layer "F.SilkS")
+		)
+		(fp_line
+			(start 6.6 1.5)
+			(end -1.5 1.5)
+			(stroke
+				(width 0.12)
+				(type solid)
+			)
+			(layer "F.SilkS")
+		)
+		(fp_line
+			(start 6.6 1.5)
+			(end 6.6 -1.5)
+			(stroke
+				(width 0.12)
+				(type solid)
+			)
+			(layer "F.SilkS")
+		)
+		(fp_line
+			(start -1.8 -1.8)
+			(end -1.8 1.8)
+			(stroke
+				(width 0.05)
+				(type solid)
+			)
+			(layer "F.CrtYd")
+		)
+		(fp_line
+			(start -1.8 -1.8)
+			(end 6.88 -1.8)
+			(stroke
+				(width 0.05)
+				(type solid)
+			)
+			(layer "F.CrtYd")
+		)
+		(fp_line
+			(start 6.88 1.8)
+			(end -1.8 1.8)
+			(stroke
+				(width 0.05)
+				(type solid)
+			)
+			(layer "F.CrtYd")
+		)
+		(fp_line
+			(start 6.88 1.8)
+			(end 6.88 -1.8)
+			(stroke
+				(width 0.05)
+				(type solid)
+			)
+			(layer "F.CrtYd")
+		)
+		(fp_line
+			(start 5.08 0)
+			(end 0 0)
+			(stroke
+				(width 0.1)
+				(type solid)
+			)
+			(layer "F.Fab")
+		)
+		(fp_text user "${REFERENCE}"
+			(at 2.54 0 0)
+			(layer "F.Fab")
+			(effects
+				(font
+					(size 1 1)
+					(thickness 0.15)
+				)
+			)
+		)
+		(pad "1" thru_hole roundrect
+			(at 0 0)
+			(size 2.6 2.6)
+			(drill 1.3)
+			(layers "*.Cu" "*.Mask")
+			(remove_unused_layers no)
+			(roundrect_rratio 0.25)
+			(net "/SYS_SWDIO")
+			(pinfunction "1_1")
+			(pintype "passive")
+		)
+		(pad "2" thru_hole circle
+			(at 5.08 0)
+			(size 2.6 2.6)
+			(drill 1.3)
+			(layers "*.Cu" "*.Mask")
+			(remove_unused_layers no)
+		)
+		(embedded_fonts no)
 	)
 	(footprint "Capacitor_SMD:C_0402_1005Metric"
@@
 			(remove_unused_layers no)
 			(roundrect_rratio 0.25)
-			(net "/SYS_SWDIO")
+			(net "/SYS_SWCLK")
 			(pinfunction "1_1")
 			(pintype "passive")
@@
 			(layers "*.Cu" "*.Mask")
 			(remove_unused_layers no)
-			(net "/SYS_SWCLK")
 		)
 		(embedded_fonts no)
